File: Design Files/omnixie/OMNIXIE_v1.kicad_pcb (KiCad board)
At the start: 2 copper layers, 19.1 x 31.8 mm, 43 parts, among them J2 Conn_01x04, J3 Conn_01x04, J4 USB_C_Receptacle_USB2.0_14P, Q0 Q_NMOS, Q1 Q_NMOS, Q10 Q_NMOS, Q11 Q_NMOS, Q2 Q_NMOS, Q3 Q_NMOS, Q4 Q_NMOS, Q5 Q_NMOS, Q6 Q_NMOS, Q7 Q_NMOS, Q8 Q_NMOS, Q9 Q_NMOS, U1 CH32V003F4U6

Commit message: commiting last work i did
Changed lines of the file:
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@@
 	)
 	(gr_rect
-		(start 148.95 136)
-		(end 168 104.25)
+		(start 148.95 104.25)
+		(end 168 136)
 		(stroke
 			(width 0.254)
