File: Design Files/omnixie/OMNIXIE_v1.kicad_sch (KiCad schematic)
At the start: 63 parts, among them J1 Conn_01x01, J2 Conn_01x04, J3 Conn_01x04, J4 USB_C_Receptacle_USB2.0_14P, Q0 Q_NMOS, Q1 Q_NMOS, Q10 Q_NMOS, Q100 Q_NMOS, Q11 Q_NMOS, Q2 Q_NMOS, Q3 Q_NMOS, Q4 Q_NMOS, Q5 Q_NMOS, Q6 Q_NMOS, Q7 Q_NMOS, Q8 Q_NMOS, Q9 Q_NMOS, T1 Flyback-ATB3225, U1 CH32V003F4U6, U2 4N25

Commit message: commiting last work i did
Parts:
- added R? (x2): 5.1k, symbol cnixxie:R
- added R?: 1.5k, symbol cnixxie:R
- added U?: XC6206P332MR, Package_TO_SOT_SMD:SOT-23-3, symbol Regulator_Linear:XC6206PxxxMR
- U3: value ~ -> PI4IOE5V6416ZDEX
Connections:
- net +5V: now also J4.A4 (VBUS), J4.A9 (VBUS), J4.B4 (VBUS), J4.B9 (VBUS), U?.3 (VI)
- net DIG_0: now also U3.1 (IO0_0)
- net DIG_1: now also U3.2 (IO0_1)
- net DIG_2: now also U3.3 (IO0_2)
- net DIG_3: now also U3.4 (IO0_3)
- net DIG_4: now also U3.5 (IO0_4)
- net DIG_5: now also U3.6 (IO0_5)
- net DIG_6: now also U3.7 (IO0_6)
- net DIG_7: now also U3.8 (IO0_7)
- net DIG_8: now also U3.10 (IO1_0)
- net DIG_9: now also U3.11 (IO1_1)
- net DIG_AUX: now also U3.13 (IO1_3)
- net DIG_DP: now also U3.12 (IO1_2)
- net GND: now also J2.4 (Pin_4), J3.4 (Pin_4), J4.A1 (GND), J4.A12 (GND), J4.B1 (GND), J4.B12 (GND), J4.S1 (SHIELD), U3.18 (ADDR), U3.9 (VSS), R?.1, R?.2, U?.1 (GND)
- net I2C_SCL: now reaches U3.19 (SCL)
- net I2C_SCL: now also J2.2 (Pin_2), J3.2 (Pin_2)
- net I2C_SDA: now reaches U3.20 (SDA)
- net I2C_SDA: now also J2.1 (Pin_1), J3.1 (Pin_1)
- net +3V3: now reaches U3.21 (VDD_P)
- net +3V3: now also J2.3 (Pin_3), J3.3 (Pin_3), U3.23 (VDD_I2C), U?.2 (VO)
- net D+: now reaches U1.17 (PD3/A4/T2CH2/AETR/UCTS/T1CH4)
- net D+: now also J4.A6 (D+), J4.B6 (D+)
- net D-: now reaches U1.18 (PD4/A7/UCK/T2CH1ETR/OPO/T1CH4ETR)
- net D-: now also J4.A7 (D-), J4.B7 (D-), R?.1
- net DPU: now reaches U1.19 (PD5/A5/UTX/T2CH4/URX)
- net DPU: now also R?.2
- net at J4.A5 (CC1): now also R?.1
- net at J4.B5 (CC2): now also R?.2
Other:
- moved on the sheet: C1, D1, FID1, FID2, FID3, FID4, H1, H2, H3, H4, J1, J2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
