File: omnixie/omnixie_v1.kicad_sch (KiCad schematic)
At the start: 67 parts, among them J1 Conn_01x01, J2 Conn_01x04, J3 Conn_01x04, J4 USB_C_Receptacle_USB2.0_14P, Q0 Q_NMOS, Q1 Q_NMOS, Q10 Q_NMOS, Q100 Q_NMOS, Q11 Q_NMOS, Q2 Q_NMOS, Q3 Q_NMOS, Q4 Q_NMOS, Q5 Q_NMOS, Q6 Q_NMOS, Q7 Q_NMOS, Q8 Q_NMOS, Q9 Q_NMOS, T1 Flyback-ATB3225, U1 CH32V003F4U6, U2 4N25, U3 PI4IOE5V6416ZDEX

Commit message: changed folder names, started bom
Parts:
- removed JP1, JP2: TH_THERM_JMP, Jumper:SolderJumper-2_P1.3mm_Open_RoundedPad1.0x1.5mm, symbol MASTER_SYMBOLS:SolderJumper_2_Open
- added C?: C, symbol Device:C
- added D?: D, symbol Device:D
- added Q?: Q_NMOS, symbol Transistor_FET:Q_NMOS_GSD
- added R? (x7): R, symbol cnixxie:R
- added T?: Flyback-ATB3225, Flyback-ATB3225:Flyback-ATB3225, symbol cnixxie:Flyback-ATB3225
- added TP? (x2): IOUTSENSE, symbol Connector:TestPoint
- added TP?: VOUTPUT, symbol Connector:TestPoint
- added TP?: GATE, symbol Connector:TestPoint
- added TP?: VFB, symbol Connector:TestPoint
- added TP? (x2): IINSENSE, symbol Connector:TestPoint
- added TP?: VD, symbol Connector:TestPoint
- added TP?: VINPUT, symbol Connector:TestPoint
Connections:
- net +5V: now also R?.1, R?.1, T?.1, T?.2, TP?.1, TP?.1; no longer TP1.1
- net EXT_GATE: now also Q100.1 (G), R10.1, TP5.1
- net GND: now also C?.2, Q?.2 (S), R?.2, R?.2
- net HIGHVOLTAGE: now also R?.1, R?.1, TP?.1; no longer C1.1, D1.1 (K), R8.1, TP3.1
- net I2C_SCL: now also U1.10 (PC3/T1CH3/T1CHIN/UCTS)
- net I2C_SDA: now also U1.9 (PC2/SCL/URTS/T1BKIN/AETR/T2CH2/T1ETR)
- net INT_GATE: now also Q?.1 (G), R?.1, TP?.1
- new net: R?.2, TP?.1
- new net: C1.1, D1.1 (K), R?.2, TP?.1
- new net: R8.1, R?.1, TP3.1
- new net: R?.2, TP1.1
- new net: D?.2 (A), T?.3, TP?.1
- new net: Q?.3 (D), T?.4
- new net FEEDBACK: R?.1, R?.2, TP?.1
- new net IOUTSENSE: C?.1, D?.1 (K), R?.2, TP?.1
Other:
- note added: "For control internally"
- note added: "For dev and experimentation"
- moved on the sheet: C1, D1, J1, Q100, R10, R8, R9, T1, TP1, TP2, TP3, TP4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
