File: kicad_projects/Production_Version/omnixie_v1.kicad_sch (KiCad schematic)
At the start: 82 parts, among them J1 Conn_01x10, J2 SM04B-SRSS-TB, J3 SM04B-SRSS-TB, J4 USB4105-GF-A, J5 Conn_01x04, J6 Conn_01x02, J8 IL-WX-16S-VF-B-E1000E, Q0 BSS123, Q1 BSS123, Q10 BSS123, Q11 BSS123, Q12 IPN50R1K4CEATMA1, Q2 BSS123, Q3 BSS123, Q4 BSS123, Q5 BSS123, Q6 BSS123, Q7 BSS123, Q8 BSS123, Q9 BSS123, T1 ATB322515-0110, U1 CH32V003F4U6, U3 PI4IOE5V6416ZDEX, U4 XC6206P332MR

Commit message: separated proto from production version with actual footprints
Parts:
- FID10, FID11, FID12, FID13, FID14, FID15, FID9: now not fitted
- TP10: now not fitted; now left out of the parts list
Connections:
- net +3V3: no longer J5.3 (Pin_3)
- net +3V3_JUMP: now reaches JP4.2 (B), U3.21 (VDD_P), U3.23 (VDD_I2C)
- net +3V3_JUMP: now also J5.3 (Pin_3)
Other:
- moved on the sheet: TP6
Changed lines of the file:
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@@
 	(text "Get a good list going for every part to buy including the little pins for smaller nixies\nAnd what I'm anticipating on putting on the board. Maybe change footprint to a footprint that I have or get some additional sized resistors with numbers on them"
 		(exclude_from_sim no)
-		(at 15.24 267.462 0)
+		(at -91.186 269.494 0)
 		(effects
 			(font
@@
 	)
 	(junction
+		(at 279.4 40.64)
+		(diameter 0)
+		(color 0 0 0 0)
+	)
+	(junction
 		(at 39.37 85.09)
 		(diameter 0)
@@
 	(wire
 		(pts
+			(xy 91.44 149.86) (xy 91.44 152.4)
+		)
+		(stroke
+			(width 0)
+			(type default)
+		)
+	)
+	(wire
+		(pts
 			(xy 262.89 88.9) (xy 262.89 91.44)
 		)
@@
 	(wire
 		(pts
-			(xy 340.36 50.8) (xy 354.33 50.8)
+			(xy 337.82 50.8) (xy 354.33 50.8)
 		)
 		(stroke
@@
 	)
 	(label "VIN_1"
-		(at 93.98 152.4 0)
+		(at 92.71 152.4 0)
 		(effects
 			(font
@@
 	)
 	(symbol
+		(lib_id "power:+5V")
+		(at 337.82 50.8 0)
+		(unit 1)
+		(exclude_from_sim no)
+		(in_bom yes)
+		(on_board yes)
+		(dnp no)
+		(property "Reference" "#PWR045"
+			(at 337.82 54.61 0)
+			(effects
+				(font
+					(size 1.27 1.27)
+				)
+				(hide yes)
+			)
+		)
+		(property "Value" "+3V3_JUMP"
+			(at 337.566 46.99 0)
+			(effects
+				(font
+					(size 1.27 1.27)
+				)
+			)
+		)
+		(property "Footprint" ""
+			(at 337.82 50.8 0)
+			(effects
+				(font
+					(size 1.27 1.27)
+				)
+				(hide yes)
+			)
+		)
+		(property "Datasheet" ""
+			(at 337.82 50.8 0)
+			(effects
+				(font
+					(size 1.27 1.27)
+				)
+				(hide yes)
+			)
+		)
+		(property "Description" "Power symbol creates a global label with name \"+5V\""
+			(at 337.82 50.8 0)
+			(effects
+				(font
+					(size 1.27 1.27)
+				)
+				(hide yes)
+			)
+		)
+		(pin "1"
+		)
+		(instances
+			(project "omnixie_v1"
+				(path "/7791313b-9c26-4810-8a43-0e3a20909b33"
+					(reference "#PWR045")
+					(unit 1)
+				)
+			)
+		)
+	)
+	(symbol
 		(lib_id "MASTER_SYMBOLS:Fiducial")
 		(at 212.09 129.54 0)
@@
 		(exclude_from_sim no)
 		(in_bom no)
-		(on_board yes)
-		(dnp no)
+		(on_board no)
+		(dnp yes)
 		(fields_autoplaced yes)
 		(property "Reference" "FID10"
@@
 		(exclude_from_sim no)
 		(in_bom no)
-		(on_board yes)
-		(dnp no)
+		(on_board no)
+		(dnp yes)
 		(fields_autoplaced yes)
 		(property "Reference" "FID14"
@@
 		(exclude_from_sim no)
 		(in_bom no)
-		(on_board yes)
-		(dnp no)
+		(on_board no)
+		(dnp yes)
 		(fields_autoplaced yes)
 		(property "Reference" "FID9"
@@
 	)
 	(symbol
+		(lib_id "power:+5V")
+		(at 279.4 40.64 0)
+		(unit 1)
+		(exclude_from_sim no)
+		(in_bom yes)
+		(on_board yes)
+		(dnp no)
+		(property "Reference" "#PWR034"
+			(at 279.4 44.45 0)
+			(effects
+				(font
+					(size 1.27 1.27)
+				)
+				(hide yes)
+			)
+		)
+		(property "Value" "+3V3_JUMP"
+			(at 279.146 36.83 0)
+			(effects
+				(font
+					(size 1.27 1.27)
+				)
+			)
+		)
+		(property "Footprint" ""
+			(at 279.4 40.64 0)
+			(effects
+				(font
+					(size 1.27 1.27)
+				)
+				(hide yes)
+			)
+		)
+		(property "Datasheet" ""
+			(at 279.4 40.64 0)
+			(effects
+				(font
+					(size 1.27 1.27)
+				)
+				(hide yes)
+			)
+		)
+		(property "Description" "Power symbol creates a global label with name \"+5V\""
+			(at 279.4 40.64 0)
+			(effects
+				(font
+					(size 1.27 1.27)
+				)
+				(hide yes)
+			)
+		)
+		(pin "1"
+		)
+		(instances
+			(project "omnixie_v1"
+				(path "/7791313b-9c26-4810-8a43-0e3a20909b33"
+					(reference "#PWR034")
+					(unit 1)
+				)
+			)
+		)
+	)
+	(symbol
 		(lib_id "cnixxie:Flyback-ATB3225")
 		(at 100.33 160.02 270)
@@
 		(exclude_from_sim no)
 		(in_bom no)
-		(on_board yes)
-		(dnp no)
+		(on_board no)
+		(dnp yes)
 		(fields_autoplaced yes)
 		(property "Reference" "FID12"
@@
 		(exclude_from_sim no)
 		(in_bom no)
-		(on_board yes)
-		(dnp no)
+		(on_board no)
+		(dnp yes)
 		(fields_autoplaced yes)
 		(property "Reference" "FID11"
@@
 		(exclude_from_sim no)
 		(in_bom no)
-		(on_board yes)
-		(dnp no)
+		(on_board no)
+		(dnp yes)
 		(fields_autoplaced yes)
 		(property "Reference" "FID13"
@@
 	)
 	(symbol
-		(lib_id "power:+5V")
-		(at 340.36 50.8 0)
-		(unit 1)
-		(exclude_from_sim no)
-		(in_bom yes)
-		(on_board yes)
-		(dnp no)
-		(property "Reference" "#PWR039"
-			(at 340.36 54.61 0)
-			(effects
-				(font
-					(size 1.27 1.27)
-				)
-				(hide yes)
-			)
-		)
-		(property "Value" "+3V3"
-			(at 340.106 46.99 0)
-			(effects
-				(font
-					(size 1.27 1.27)
-				)
-			)
-		)
-		(property "Footprint" ""
-			(at 340.36 50.8 0)
-			(effects
-				(font
-					(size 1.27 1.27)
-				)
-				(hide yes)
-			)
-		)
-		(property "Datasheet" ""
-			(at 340.36 50.8 0)
-			(effects
-				(font
-					(size 1.27 1.27)
-				)
-				(hide yes)
-			)
-		)
-		(property "Description" "Power symbol creates a global label with name \"+5V\""
-			(at 340.36 50.8 0)
-			(effects
-				(font
-					(size 1.27 1.27)
-				)
-				(hide yes)
-			)
-		)
-		(pin "1"
-		)
-		(instances
-			(project "omnixie_v1"
-				(path "/7791313b-9c26-4810-8a43-0e3a20909b33"
-					(reference "#PWR039")
-					(unit 1)
-				)
-			)
-		)
-	)
-	(symbol
 		(lib_id "Connector:TestPoint")
 		(at 74.93 152.4 0)
 		(unit 1)
 		(exclude_from_sim no)
-		(in_bom yes)
-		(on_board yes)
-		(dnp no)
+		(in_bom no)
+		(on_board no)
+		(dnp yes)
 		(property "Reference" "TP10"
 			(at 74.93 147.066 0)
@@
 	(symbol
 		(lib_id "Connector:TestPoint")
-		(at 91.44 152.4 0)
+		(at 91.44 149.86 0)
 		(unit 1)
 		(exclude_from_sim no)
@@
 		(dnp no)
 		(property "Reference" "TP6"
-			(at 91.44 146.558 0)
+			(at 91.44 144.018 0)
 			(effects
 				(font
@@
 		)
 		(property "Value" "5005"
-			(at 91.186 144.018 0)
+			(at 91.186 141.478 0)
 			(effects
 				(font
@@
 		)
 		(property "Footprint" "TestPoint:TestPoint_Keystone_5005-5009_Compact"
-			(at 96.52 152.4 0)
+			(at 96.52 149.86 0)
 			(effects
 				(font
@@
 		)
 		(property "Datasheet" "~"
-			(at 96.52 152.4 0)
+			(at 96.52 149.86 0)
 			(effects
 				(font
@@
 		)
 		(property "Description" "IINSENSE"
-			(at 91.44 152.4 0)
+			(at 91.44 149.86 0)
 			(effects
 				(font
@@
 		(exclude_from_sim no)
 		(in_bom no)
-		(on_board yes)
-		(dnp no)
+		(on_board no)
+		(dnp yes)
 		(fields_autoplaced yes)
 		(property "Reference" "FID15"
