File: kicad_projects/omnixie_proto_v1/omnixie_v1.kicad_pcb (KiCad board)
At the start: 2 copper layers, 35.6 x 33 mm, 53 parts, among them J1 Conn_01x10, J4 USB4105-GF-A, J5 Conn_01x04, J6 Conn_01x02, J8 IL-WX-16S-VF-B-E1000E, Q0 BSS123, Q1 BSS123, Q10 BSS123, Q11 BSS123, Q12 IPN50R1K4CEATMA1, Q2 BSS123, Q3 BSS123, Q4 BSS123, Q5 BSS123, Q6 BSS123, Q7 BSS123, Q8 BSS123, Q9 BSS123, T1 ATB322515-0110, U1 CH32V003F4U6, U3 PI4IOE5V6416ZDEX, U4 XC6206P332MR

Commit message: p much done, no nixie hat board though
Parts:
- C3, C4, C5: footprint Capacitor_SMD:C_0603_1608Metric -> Capacitor_SMD:C_0805_2012Metric
- Q0, Q1, Q10, Q11, Q2, Q3, Q4, Q5, Q6, Q7, Q8, Q9, U4: footprint Package_TO_SOT_SMD:SOT-23-3 -> OMNIXIE:SOT-23-3-NO_SILK
- R10, R16: footprint Resistor_SMD:R_0402_1005Metric -> Resistor_SMD:R_0805_2012Metric
- R11, R12, R13, R14: footprint Resistor_SMD:R_0603_1608Metric -> Resistor_SMD:R_0805_2012Metric
- R15, R7, R8, R9: footprint Resistor_SMD:R_0402_1005Metric_Pad0.72x0.64mm_HandSolder -> Resistor_SMD:R_0805_2012Metric
- U3: footprint Package_DFN_QFN:TQFN-24-1EP_4x4mm_P0.5mm_EP2.1x2.1mm_ThermalVias -> OMNIXIE:PI4IOE5V6416ZDEX-TQFN24
- moved R14 3.97 mm to (161.1, 92.1), turned to -90 degrees
- moved ? 3.26 mm to (123.0, 83.9)
- moved R6 1.66 mm to (138.6, 72.2)
- moved R15 1.27 mm to (158.1, 89.9)
- moved R12 0.99 mm to (145.5, 68.3)
- moved C4 0.93 mm to (153.7, 88.1)
- moved R5 0.84 mm to (138.7, 76.9)
- moved R16 0.84 mm to (158.4, 82.5)
- moved C5 0.66 mm to (148.5, 82.3)
- moved R8 0.59 mm to (158.3, 87.9)
- moved D3 0.59 mm to (153.2, 76.9)
- moved R9 0.55 mm to (158.3, 85.9)
- moved R13 0.51 mm to (161.5, 84.8)
- moved R7 0.48 mm to (136.6, 77.1)
- moved TP6 0.46 mm to (151.1, 74.2)
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Routing:
- net GND: track 48.1 -> 25.1 mm, vias 25 -> 57
- net +3V3: track 21.1 -> 14.4 mm
- net +5V_FLY: track 6.29 -> 0.00 mm
- net Net-(Q12-D): track 6.09 -> 0.00 mm
- net /D_2: track 9.69 -> 3.88 mm
- net /HV_1: track 15.4 -> 9.82 mm
- net /CC2: track 8.27 -> 12.9 mm
- net +3V3_JUMP: track 28.9 -> 25.0 mm
- net /D_1: track 6.59 -> 3.38 mm
- net HV_SW: track 35.2 -> 37.2 mm
- net DPU: track 2.07 -> 3.86 mm
- net /D-_1: track 3.52 -> 5.08 mm
- net CATHDP: track 5.33 -> 6.68 mm
- net PC6: track 22.9 -> 24.1 mm
- net PC5: track 19.2 -> 20.3 mm
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- added copper zone on F.Cu, net +3V3_JUMP
- added copper zone on F.Cu, net /D_1
- added copper zone on F.Cu, net /D_2
- added copper zone on F.Cu, net /HV_1
- added copper zone on F.Cu, net Net-(Q12-D)
Other:
- board text added: "+3V3"
- board text added: "+5V"
- board text added: "0"
- board text added: "1"
- board text added: "2"
- board text added: "3"
- board text added: "4"
- board text added: "5"
- board text added: "6"
- board text added: "7"
- board text added: "8"
- board text added: "9"
- board text added: "AUX"
- board text added: "D1_ANODE"
- board text added: "D1_CATHODE"
- board text added: "DP"
- board text added: "FEEDBACK"
- board text added: "GND"
- board text added: "HIGH VOLTAGE!"
- board text added: "PA1"
- board text added: "PA2"
- board text added: "PC0"
- board text added: "PC1"
- board text added: "PC5"
- board text added: "PC6"
- board text added: "PD0"
- board text added: "PD2"
- board text added: "PD6"
- board text added: "PD7"
- board text added: "PROGRAM"
- board text added: "R6 ANODE RESISTOR"
- board text added: "SCL"
- board text added: "SDA"
- board text added: "SW"
- board text added: "VIN"
