File: kicad_projects/omnixie_proto_v1/omnixie_v1.kicad_sch (KiCad schematic)
At the start: 82 parts, among them J1 Conn_01x10, J2 SM04B-SRSS-TB, J3 SM04B-SRSS-TB, J4 USB4105-GF-A, J5 Conn_01x04, J6 Conn_01x02, J8 IL-WX-16S-VF-B-E1000E, Q0 BSS123, Q1 BSS123, Q10 BSS123, Q11 BSS123, Q12 IPN50R1K4CEATMA1, Q2 BSS123, Q3 BSS123, Q4 BSS123, Q5 BSS123, Q6 BSS123, Q7 BSS123, Q8 BSS123, Q9 BSS123, T1 ATB322515-0110, U1 CH32V003F4U6, U3 PI4IOE5V6416ZDEX, U4 XC6206P332MR

Commit message: p much done, no nixie hat board though
Parts:
- C3, C4, C5: footprint Capacitor_SMD:C_0603_1608Metric -> Capacitor_SMD:C_0805_2012Metric
- Q0, Q1, Q10, Q11, Q2, Q3, Q4, Q5, Q6, Q7, Q8, Q9, U4: footprint Package_TO_SOT_SMD:SOT-23-3 -> OMNIXIE:SOT-23-3-NO_SILK
- R10, R16: footprint Resistor_SMD:R_0402_1005Metric -> Resistor_SMD:R_0805_2012Metric
- R11, R12, R13, R14: footprint Resistor_SMD:R_0603_1608Metric -> Resistor_SMD:R_0805_2012Metric
- R15, R7, R8, R9: footprint Resistor_SMD:R_0402_1005Metric_Pad0.72x0.64mm_HandSolder -> Resistor_SMD:R_0805_2012Metric
- U3: footprint Package_DFN_QFN:TQFN-24-1EP_4x4mm_P0.5mm_EP2.1x2.1mm_ThermalVias -> OMNIXIE:PI4IOE5V6416ZDEX-TQFN24
Other:
- note removed: "Get a good list going for every part to buy including the little pins for smaller nixies And what I'm anticipating on putting on the board. Maybe change footprint to a footprint that I have or get some additional sized resistors with numbers on them"
Changed lines of the file:
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@@
 		)
 	)
-	(text "Get a good list going for every part to buy including the little pins for smaller nixies\nAnd what I'm anticipating on putting on the board. Maybe change footprint to a footprint that I have or get some additional sized resistors with numbers on them"
-		(exclude_from_sim no)
-		(at -91.186 269.494 0)
-		(effects
-			(font
-				(size 1.27 1.27)
-				(thickness 0.3556)
-				(bold yes)
-				(italic yes)
-			)
-			(justify left)
-		)
-	)
 	(text "Likely remove pinout on the right side of board"
 		(exclude_from_sim no)
@@
 			)
 		)
-		(property "Footprint" "Package_TO_SOT_SMD:SOT-23-3"
+		(property "Footprint" "OMNIXIE:SOT-23-3-NO_SILK"
 			(at 261.62 232.41 0)
 			(effects
@@
 			)
 		)
-		(property "Datasheet" "~"
+		(property "Datasheet" ""
 			(at 256.54 234.95 0)
 			(effects
@@
 			)
 		)
-		(property "Description" "N-MOSFET transistor, gate/source/drain"
+		(property "Description" ""
 			(at 256.54 234.95 0)
 			(effects
@@
 			)
 		)
-		(property "Footprint" "Package_DFN_QFN:TQFN-24-1EP_4x4mm_P0.5mm_EP2.1x2.1mm_ThermalVias"
+		(property "Footprint" "OMNIXIE:PI4IOE5V6416ZDEX-TQFN24"
 			(at 278.13 68.58 0)
 			(effects
@@
 			)
 		)
-		(property "Footprint" "Capacitor_SMD:C_0603_1608Metric"
+		(property "Footprint" "Capacitor_SMD:C_0805_2012Metric"
 			(at 67.0052 160.02 0)
 			(effects
@@
 			)
 		)
-		(property "Footprint" "Package_TO_SOT_SMD:SOT-23-3"
+		(property "Footprint" "OMNIXIE:SOT-23-3-NO_SILK"
 			(at 232.41 232.41 0)
 			(effects
@@
 			)
 		)
-		(property "Datasheet" "~"
+		(property "Datasheet" ""
 			(at 227.33 234.95 0)
 			(effects
@@
 			)
 		)
-		(property "Description" "N-MOSFET transistor, gate/source/drain"
+		(property "Description" ""
 			(at 227.33 234.95 0)
 			(effects
@@
 			)
 		)
-		(property "Footprint" "Package_TO_SOT_SMD:SOT-23-3"
+		(property "Footprint" "OMNIXIE:SOT-23-3-NO_SILK"
 			(at 135.89 232.41 0)
 			(effects
@@
 			)
 		)
-		(property "Datasheet" "~"
+		(property "Datasheet" ""
 			(at 130.81 234.95 0)
 			(effects
@@
 			)
 		)
-		(property "Description" "N-MOSFET transistor, gate/source/drain"
+		(property "Description" ""
 			(at 130.81 234.95 0)
 			(effects
@@
 			)
 		)
-		(property "Footprint" "Package_TO_SOT_SMD:SOT-23-3"
+		(property "Footprint" "OMNIXIE:SOT-23-3-NO_SILK"
 			(at 200.66 232.41 0)
 			(effects
@@
 			)
 		)
-		(property "Datasheet" "~"
+		(property "Datasheet" ""
 			(at 195.58 234.95 0)
 			(effects
@@
 			)
 		)
-		(property "Description" "N-MOSFET transistor, gate/source/drain"
+		(property "Description" ""
 			(at 195.58 234.95 0)
 			(effects
@@
 			)
 		)
-		(property "Footprint" "Package_TO_SOT_SMD:SOT-23-3"
+		(property "Footprint" "OMNIXIE:SOT-23-3-NO_SILK"
 			(at 323.85 232.41 0)
 			(effects
@@
 			)
 		)
-		(property "Datasheet" "~"
+		(property "Datasheet" ""
 			(at 318.77 234.95 0)
 			(effects
@@
 			)
 		)
-		(property "Description" "N-MOSFET transistor, gate/source/drain"
+		(property "Description" ""
 			(at 318.77 234.95 0)
 			(effects
@@
 			)
 		)
-		(property "Footprint" "Resistor_SMD:R_0603_1608Metric"
+		(property "Footprint" "Resistor_SMD:R_0805_2012Metric"
 			(at 88.392 184.15 90)
 			(effects
@@
 			)
 		)
-		(property "Footprint" "Resistor_SMD:R_0603_1608Metric"
+		(property "Footprint" "Resistor_SMD:R_0805_2012Metric"
 			(at 130.302 181.61 90)
 			(effects
@@
 			)
 		)
-		(property "Footprint" "Package_TO_SOT_SMD:SOT-23-3"
+		(property "Footprint" "OMNIXIE:SOT-23-3-NO_SILK"
 			(at 355.6 233.68 0)
 			(effects
@@
 			)
 		)
-		(property "Datasheet" "~"
+		(property "Datasheet" ""
 			(at 350.52 236.22 0)
 			(effects
@@
 			)
 		)
-		(property "Description" "N-MOSFET transistor, gate/source/drain"
+		(property "Description" ""
 			(at 350.52 236.22 0)
 			(effects
@@
 			)
 		)
-		(property "Footprint" "Package_TO_SOT_SMD:SOT-23-3"
+		(property "Footprint" "OMNIXIE:SOT-23-3-NO_SILK"
 			(at 384.81 233.68 0)
 			(effects
@@
 			)
 		)
-		(property "Datasheet" "~"
+		(property "Datasheet" ""
 			(at 379.73 236.22 0)
 			(effects
@@
 			)
 		)
-		(property "Description" "N-MOSFET transistor, gate/source/drain"
+		(property "Description" ""
 			(at 379.73 236.22 0)
 			(effects
@@
 			)
 		)
-		(property "Footprint" "Package_TO_SOT_SMD:SOT-23-3"
+		(property "Footprint" "OMNIXIE:SOT-23-3-NO_SILK"
 			(at 168.91 232.41 0)
 			(effects
@@
 			)
 		)
-		(property "Datasheet" "~"
+		(property "Datasheet" ""
 			(at 163.83 234.95 0)
 			(effects
@@
 			)
 		)
-		(property "Description" "N-MOSFET transistor, gate/source/drain"
+		(property "Description" ""
 			(at 163.83 234.95 0)
 			(effects
@@
 			)
 		)
-		(property "Footprint" "Resistor_SMD:R_0402_1005Metric_Pad0.72x0.64mm_HandSolder"
+		(property "Footprint" "Resistor_SMD:R_0805_2012Metric"
 			(at 232.41 35.052 90)
 			(effects
@@
 			)
 		)
-		(property "Footprint" "Resistor_SMD:R_0402_1005Metric_Pad0.72x0.64mm_HandSolder"
+		(property "Footprint" "Resistor_SMD:R_0805_2012Metric"
 			(at 130.302 171.45 90)
 			(effects
@@
 			)
 		)
-		(property "Footprint" "Resistor_SMD:R_0603_1608Metric"
+		(property "Footprint" "Resistor_SMD:R_0805_2012Metric"
 			(at 68.58 51.308 90)
 			(effects
@@
 			)
 		)
-		(property "Footprint" "Resistor_SMD:R_0402_1005Metric"
+		(property "Footprint" "Resistor_SMD:R_0805_2012Metric"
 			(at 132.08 101.6 0)
 			(effects
@@
 			)
 		)
-		(property "Footprint" "Resistor_SMD:R_0402_1005Metric_Pad0.72x0.64mm_HandSolder"
+		(property "Footprint" "Resistor_SMD:R_0805_2012Metric"
 			(at 226.822 29.21 90)
 			(effects
@@
 			)
 		)
-		(property "Footprint" "Package_TO_SOT_SMD:SOT-23-3"
+		(property "Footprint" "OMNIXIE:SOT-23-3-NO_SILK"
 			(at 74.93 232.41 0)
 			(effects
@@
 			)
 		)
-		(property "Datasheet" "~"
+		(property "Datasheet" ""
 			(at 69.85 234.95 0)
 			(effects
@@
 			)
 		)
-		(property "Description" "N-MOSFET transistor, gate/source/drain"
+		(property "Description" ""
 			(at 69.85 234.95 0)
 			(effects
@@
 			)
 		)
-		(property "Footprint" "Capacitor_SMD:C_0603_1608Metric"
+		(property "Footprint" "Capacitor_SMD:C_0805_2012Metric"
 			(at 100.0252 66.04 0)
 			(effects
@@
 			)
 		)
-		(property "Footprint" "Package_TO_SOT_SMD:SOT-23-3"
+		(property "Footprint" "OMNIXIE:SOT-23-3-NO_SILK"
 			(at 43.18 232.41 0)
 			(effects
@@
 			)
 		)
-		(property "Datasheet" "~"
+		(property "Datasheet" ""
 			(at 38.1 234.95 0)
 			(effects
@@
 			)
 		)
-		(property "Description" "N-MOSFET transistor, gate/source/drain"
+		(property "Description" ""
 			(at 38.1 234.95 0)
 			(effects
@@
 			)
 		)
-		(property "Footprint" "Package_TO_SOT_SMD:SOT-23-3"
+		(property "Footprint" "OMNIXIE:SOT-23-3-NO_SILK"
 			(at 292.1 232.41 0)
 			(effects
@@
 			)
 		)
-		(property "Datasheet" "~"
+		(property "Datasheet" ""
 			(at 287.02 234.95 0)
 			(effects
@@
 			)
 		)
-		(property "Description" "N-MOSFET transistor, gate/source/drain"
+		(property "Description" ""
 			(at 287.02 234.95 0)
 			(effects
@@
 			)
 		)
-		(property "Footprint" "Resistor_SMD:R_0603_1608Metric"
+		(property "Footprint" "Resistor_SMD:R_0805_2012Metric"
 			(at 68.58 50.292 90)
 			(effects
@@
 			)
 		)
-		(property "Footprint" "Resistor_SMD:R_0402_1005Metric_Pad0.72x0.64mm_HandSolder"
+		(property "Footprint" "Resistor_SMD:R_0805_2012Metric"
 			(at 232.41 38.862 90)
 			(effects
@@
 			)
 		)
-		(property "Footprint" "Capacitor_SMD:C_0603_1608Metric"
+		(property "Footprint" "Capacitor_SMD:C_0805_2012Metric"
 			(at 86.0552 101.6 0)
 			(effects
@@
 			)
 		)
-		(property "Footprint" "Resistor_SMD:R_0402_1005Metric"
+		(property "Footprint" "Resistor_SMD:R_0805_2012Metric"
 			(at 115.57 101.6 0)
 			(effects
@@
 			)
 		)
-		(property "Footprint" "Package_TO_SOT_SMD:SOT-23-3"
+		(property "Footprint" "OMNIXIE:SOT-23-3-NO_SILK"
 			(at 73.66 88.265 0)
 			(effects
@@
 			)
 		)
-		(property "Datasheet" "https://www.torexsemi.com/file/xc6206/XC6206.pdf"
+		(property "Datasheet" ""
 			(at 73.66 93.98 0)
 			(effects
@@
 			)
 		)
-		(property "Description" "Positive 60-250mA Low Dropout Regulator, Fixed Output, SOT-23"
+		(property "Description" ""
 			(at 73.66 93.98 0)
 			(effects
@@
 			)
 		)
-		(property "Footprint" "Package_TO_SOT_SMD:SOT-23-3"
+		(property "Footprint" "OMNIXIE:SOT-23-3-NO_SILK"
 			(at 106.68 232.41 0)
 			(effects
@@
 			)
 		)
-		(property "Datasheet" "~"
+		(property "Datasheet" ""
 			(at 101.6 234.95 0)
 			(effects
@@
 			)
 		)
-		(property "Description" "N-MOSFET transistor, gate/source/drain"
+		(property "Description" ""
 			(at 101.6 234.95 0)
 			(effects
