File: kicad_projects/omnixieTestHAT_v0.2/omnixieHAT_v0_2.kicad_pcb (KiCad board)
At the start: 2 copper layers, 91.4 x 55.9 mm, 9 parts, among them J1 IL-WX-16PB-VF-B-E1000E

Commit message: board bringup starting now
Parts:
- added TP1: 9, Connector_PinHeader_2.54mm:PinHeader_1x01_P2.54mm_Vertical, F.Cu at (145.6, 119.6)
- added TP2: 1, Connector_PinHeader_2.54mm:PinHeader_1x01_P2.54mm_Vertical, F.Cu at (155.4, 108.8)
- N1: footprint NIXIE:IN-1_NIXIE_v1 -> OMNIXIE:IN-1_NIXIE_v1
- N4: footprint NIXIE:IN-12A Nixie -> OMNIXIE:IN-12A Nixie
Routing:
- net CATH1: track 191.7 -> 197.8 mm
- net CATH9: track 159.0 -> 163.4 mm
- net CATH3: track 163.6 -> 167.0 mm
- net CATH7: track 149.2 -> 152.1 mm
- net HIGHVOLTAGE: track 221.9 -> 224.4 mm
- net CATH0: track 212.7 -> 215.0 mm
- net CATH6: track 165.4 -> 166.8 mm
- net CATH8: track 182.6 -> 183.9 mm
- net CATH4: track 167.1 -> 168.3 mm
- net CATH5: track 130.0 -> 130.9 mm
- net CATH2: track 179.6 -> 180.3 mm
Other:
- board text added: "8-10-2026"
- board text added: "OmnixieHATv0.2"
- board text removed: "1-14-2025"
- board text removed: "OmnixieHAT"
