File: kicad_projects/omnixieTestHAT_v0.2/omnixieHAT_v0_2.kicad_sch (KiCad schematic)
At the start: 10 parts, among them J1 IL-WX-16PB-VF-B-E1000E, J2 Conn_02x08_Counter_Clockwise

Commit message: redlines almost done, new layout commencing
Parts:
- N1, N2, N3, N5, N6, N7: value ~ -> (none)
Other:
- note added: ">.< Double check all footprints."
- note added: ">.< Silkscreen WAY TOO SMALL to be easily legible from a reasonable distance"
- note added: ">.< Understand for the omnixie hat connector what orientation is will connect to the omnixie driver board."
- note added: "REDLINE NOTES"

Commit message: board bringup starting now
Parts:
- removed J2: Conn_02x08_Counter_Clockwise, symbol Connector_Generic:Conn_02x08_Counter_Clockwise
- added TP1: 9, Connector_PinHeader_2.54mm:PinHeader_1x01_P2.54mm_Vertical, symbol Connector:TestPoint
- added TP2: 1, Connector_PinHeader_2.54mm:PinHeader_1x01_P2.54mm_Vertical, symbol Connector:TestPoint
- N1: footprint NIXIE:IN-1_NIXIE_v1 -> OMNIXIE:IN-1_NIXIE_v1
- N4: footprint NIXIE:IN-12A Nixie -> OMNIXIE:IN-12A Nixie
Connections:
- net CATH1: now also TP2.1
- net CATH9: now also TP1.1
Other:
- note removed: ">.< Double check all footprints."
- note removed: ">.< Silkscreen WAY TOO SMALL to be easily legible from a reasonable distance"
- note removed: ">.< Understand for the omnixie hat connector what orientation is will connect to the omnixie driver board."
- note removed: "REDLINE NOTES"
