File: kicad_projects/omnixie_v0.2/omnixie_v0_2.kicad_pcb (KiCad board)
At the start: 2 copper layers, 35.6 x 33 mm, 51 parts, among them J1 Conn_01x10, J4 USB4105-GF-A, J5 Conn_01x04, J6 Conn_01x02, J8 IL-WX-16S-VF-B-E1000E, Q0 BSS123, Q1 BSS123, Q10 BSS123, Q11 BSS123, Q12 IPN50R1K4CEATMA1, Q2 BSS123, Q3 BSS123, Q4 BSS123, Q5 BSS123, Q6 BSS123, Q7 BSS123, Q8 BSS123, Q9 BSS123, T1 ATB322515-0110, U1 CH32V003F4U6, U3 PI4IOE5V6416ZDEX, U4 XC6206P332MR

Commit message: new folders for next versions
Other:
- board size 35.6 x 33 mm -> 105 x 43.2 mm

Commit message: redlines almost done, new layout commencing
Parts:
- added J2: SM04B-SRSS-TB, Connector_JST:JST_SH_SM04B-SRSS-TB_1x04-1MP_P1.00mm_Horizontal, F.Cu at (134.5, 128.0)
- added J3: SM04B-SRSS-TB, Connector_JST:JST_SH_SM04B-SRSS-TB_1x04-1MP_P1.00mm_Horizontal, F.Cu at (134.5, 135.6)
- added J7: Conn_02x08_Counter_Clockwise, Connector_PinHeader_2.54mm:PinHeader_2x08_P2.54mm_Vertical, F.Cu at (102.6, 43.4)
- added TP10: 5005, TestPoint:TestPoint_Keystone_5005-5009_Compact, F.Cu at (69.6, 96.8)
- added TP15: 5005, TestPoint:TestPoint_Keystone_5005-5009_Compact, F.Cu at (87.4, 147.6)
- added TP16: 5005, TestPoint:TestPoint_Keystone_5005-5009_Compact, F.Cu at (87.4, 152.7)
- added TP17: 5005, TestPoint:TestPoint_Keystone_5005-5009_Compact, F.Cu at (92.4, 142.6)
- added TP18: 5005, TestPoint:TestPoint_Keystone_5005-5009_Compact, F.Cu at (92.4, 147.6)
- added TP19: 5005, TestPoint:TestPoint_Keystone_5005-5009_Compact, F.Cu at (92.4, 152.7)
- added TP20: 5005, TestPoint:TestPoint_Keystone_5005-5009_Compact, F.Cu at (97.5, 142.6)
- added TP21: 5005, TestPoint:TestPoint_Keystone_5005-5009_Compact, F.Cu at (97.5, 147.6)
- added TP22: 5005, TestPoint:TestPoint_Keystone_5005-5009_Compact, F.Cu at (55.7, 53.6)
- added TP23: 5005, TestPoint:TestPoint_Keystone_5005-5009_Compact, F.Cu at (60.7, 43.5)
- added TP24: 5005, TestPoint:TestPoint_Keystone_5005-5009_Compact, F.Cu at (60.7, 48.6)
- added TP25: 5005, TestPoint:TestPoint_Keystone_5005-5009_Compact, F.Cu at (60.7, 53.6)
- C2: footprint Capacitor_SMD:C_1210_3225Metric -> Capacitor_SMD:C_1812_4532Metric_Pad1.57x3.40mm_HandSolder
- J4: footprint OMNIXIE:USB4120-03-C -> Connector_USB:USB_C_Receptacle_GCT_USB4105-xx-A_16P_TopMnt_Horizontal; moved to F.Cu
- Q12: value IPN50R1K4CEATMA1 -> STN1NK60ZL; footprint Package_TO_SOT_SMD:SOT-223-3_TabPin2 -> OMNIXIE:SOT-223-MiddlePinDrain
- R10, R16: value 10k -> 30K
- R15, R8, R9, U1: moved to F.Cu
- R3: footprint Resistor_SMD:R_0603_1608Metric -> Resistor_SMD:R_0603_1608Metric_Pad0.98x0.95mm_HandSolder
- moved R11 102.8 mm to (56.7, 111.1)
- moved J5 97.1 mm to (48.0, 43.4)
- moved TP6 95.0 mm to (67.1, 112.0)
- moved C5 93.1 mm to (61.2, 106.1)
- moved D1 93.1 mm to (53.5, 103.6)
- moved Q12 93.1 mm to (57.3, 98.2)
- moved R12 93.1 mm to (58.1, 92.1)
- moved R3 93.1 mm to (63.1, 103.6)
- moved R5 93.1 mm to (51.3, 100.7)
- moved R6 93.1 mm to (51.3, 96.1)
- moved R7 93.1 mm to (49.3, 101.0)
- moved TP11 93.1 mm to (57.4, 107.3)
- moved TP14 93.1 mm to (53.6, 90.9)
- moved TP8 93.1 mm to (51.6, 110.4)
- moved C2 93.1 mm to (53.3, 106.6)
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Connections:
- Q12 pad 2: GND -> Net-(Q12-D)
- Q12 pad 3: Net-(Q12-D) -> GND
- U1 pad 10: I2C_SCL -> PC3
- U1 pad 8: PC1 -> I2C_SDA
- U1 pad 9: I2C_SDA -> I2C_SCL
Routing:
- net /CC2: track 12.9 -> 0.00 mm, vias 1 -> 0
- net +5V: track 23.2 -> 36.1 mm, vias 3 -> 4
- net PC6: track 24.1 -> 17.5 mm
- net PC0: track 9.87 -> 3.52 mm
- net PA2: track 6.59 -> 1.34 mm
- net PD6: track 5.23 -> 0.00 mm
- net PC1: track 12.6 -> 7.70 mm
- net PD7: track 3.66 -> 0.00 mm
- net PD0: track 7.55 -> 4.00 mm
- net PC5: track 20.3 -> 17.0 mm
- net PA1: track 4.55 -> 1.50 mm
- net PD2: track 29.0 -> 26.3 mm
- net GND: track 25.1 -> 23.4 mm
- net D-: track 16.7 -> 16.0 mm
Other:
- board size 105 x 43.2 mm -> 141.4 x 79.4 mm

Commit message: board bringup starting now
Parts:
- removed TP15, TP16, TP21: 5005, TestPoint:TestPoint_Keystone_5005-5009_Compact
- added R17: JUMPER, Resistor_SMD:R_0805_2012Metric, F.Cu at (142.5, 89.4)
- moved SCL 117.5 mm to (169.9, 80.8)
- moved SDA 116.9 mm to (169.9, 85.1)
- moved J5 115.5 mm to (157.5, 80.3), turned to 0 degrees
- moved +3V3 109.7 mm to (165.6, 80.8)
- moved GND 109.5 mm to (165.6, 85.1)
- moved R7 99.9 mm to (148.3, 114.0)
- moved TP13 95.5 mm to (144.3, 114.0)
- moved R11 95.4 mm to (152.1, 114.0), turned to 90 degrees
- moved TP14 95.2 mm to (148.3, 81.8), turned to 90 degrees
- moved TP18 95.1 mm to (175.5, 101.3)
- moved J1 93.6 mm to (151.8, 119.6), turned to -90 degrees
- moved Q6 91.4 mm to (178.8, 60.5)
- moved Q10 91.1 mm to (180.1, 70.4)
- moved Q9 90.7 mm to (179.8, 66.5)
- moved Q11 87.7 mm to (174.8, 68.8)
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- renumbered TP24 to +3V3, TP17 to +3V3, D2 to +5V, TP20 to D+, TP19 to D-, TP25 to GND, TP10 to RIS1, TP22 to SCL, TP23 to SDA
Connections:
- +3V3 pad 1: +3V3_JUMP -> +3V3
- J1 pad 1: PD2 -> PD6
- J1 pad 10: PD6 -> PA1
- J1 pad 2: PC6 -> PD7
- J1 pad 3: PC5 -> PD2
- J1 pad 4: PC1 -> PC6
- J1 pad 5: PC0 -> PC5
- J1 pad 6: PD0 -> PC3
- J1 pad 7: PA2 -> PC0
- J1 pad 8: PA1 -> PD0
- J1 pad 9: PD7 -> PA2
- J5 pad 3: +3V3_JUMP -> +3V3
- J7 pad 10: CATH9 -> unconnected-(J7-Pin_10-Pad10)
- J7 pad 11: CATHDP -> unconnected-(J7-Pin_11-Pad11)
- J7 pad 12: CATHAUX -> unconnected-(J7-Pin_12-Pad12)
- J7 pad 6: CATH5 -> unconnected-(J7-Pin_6-Pad6)
- J7 pad 8: CATH7 -> unconnected-(J7-Pin_8-Pad8)
- J7 pad 9: CATH8 -> unconnected-(J7-Pin_9-Pad9)
- Q12 pad 1: HV_SW -> Net-(Q12-G)
- R12 pad 1: HV_SW -> Net-(Q12-G)
- TP14 pad 1: HV_SW -> Net-(Q12-G)
Routing:
- net +3V3: track 14.4 -> 104.6 mm, vias 3 -> 2
- net CATH6: track 6.33 -> 58.6 mm
- net /HV_1: track 10.3 -> 58.6 mm, vias 0 -> 2
- net HIGHVOLTAGE: track 22.3 -> 67.0 mm
- net GND: track 23.4 -> 66.8 mm, vias 57 -> 48
- net PA1: track 1.50 -> 42.0 mm
- net PROGRAM: track 13.6 -> 52.4 mm, vias 0 -> 1
- net PA2: track 1.34 -> 36.4 mm
- net CATH4: track 4.31 -> 35.9 mm
- net PD7: track 0.00 -> 29.2 mm, vias 0 -> 2
- net CATH3: track 8.40 -> 36.2 mm, vias 2 -> 0
- net PD0: track 4.00 -> 28.2 mm
- net CATH2: track 2.81 -> 25.4 mm
- net CATH1: track 8.32 -> 29.2 mm, vias 2 -> 0
- net PC0: track 3.52 -> 24.0 mm
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- removed copper zone on F.Cu, net +3V3
- removed copper zone on F.Cu, net +3V3_JUMP
Other:
- board size 141.4 x 79.4 mm -> 62.3 x 71.5 mm
- board text added: "8-10-2026"
- board text added: "ANODE RESISTOR"
- board text added: "D+"
- board text added: "D-"
- board text added: "G"
- board text added: "GATE"
- board text added: "HV"
- board text added: "NA DESIGN"
- board text added: "NOT APPLICABLE"
- board text added: "PC3"
- board text added: "PRGM"
- board text added: "RIS1"
- board text added: "RIS2"
- board text added: "ROS1"
- board text added: "ROS2"
- board text added: "TP18"
- board text added: "V0.2 PROTO"
- board text removed: "1-14-2025"
- board text removed: "D1_ANODE"
- board text removed: "D1_CATHODE"
- board text removed: "NICOLAS ALVAREZ"
- board text removed: "PC1"
- board text removed: "PROGRAM"
- board text removed: "R6 ANODE RESISTOR"
- board text removed: "SW"
- board text removed: "V1"
- board text removed: "VIN"
