File: kicad_projects/omnixie_v0.2/omnixie_v0_2.kicad_sch (KiCad schematic)
At the start: 67 parts, among them J1 Conn_01x10, J2 SM04B-SRSS-TB, J3 SM04B-SRSS-TB, J4 USB4105-GF-A, J5 Conn_01x04, J6 Conn_01x02, J8 IL-WX-16S-VF-B-E1000E, Q0 BSS123, Q1 BSS123, Q10 BSS123, Q11 BSS123, Q12 IPN50R1K4CEATMA1, Q2 BSS123, Q3 BSS123, Q4 BSS123, Q5 BSS123, Q6 BSS123, Q7 BSS123, Q8 BSS123, Q9 BSS123, T1 ATB322515-0110, U1 CH32V003F4U6, U3 PI4IOE5V6416ZDEX, U4 XC6206P332MR

Commit message: redlines almost done, new layout commencing
Parts:
- added J7: Conn_02x08_Counter_Clockwise, Connector_PinHeader_2.54mm:PinHeader_2x08_P2.54mm_Vertical, symbol Connector_Generic:Conn_02x08_Counter_Clockwise
- added TP15, TP16, TP17, TP18, TP19, TP20, TP21, TP22, TP23, TP24, TP25: 5005, TestPoint:TestPoint_Keystone_5005-5009_Compact, symbol Connector:TestPoint
- C2: footprint Capacitor_SMD:C_1210_3225Metric -> Capacitor_SMD:C_1812_4532Metric_Pad1.57x3.40mm_HandSolder
- J2, J3: now in the parts list
- J4: footprint OMNIXIE:USB4120-03-C -> Connector_USB:USB_C_Receptacle_GCT_USB4105-xx-A_16P_TopMnt_Horizontal
- Q12: value IPN50R1K4CEATMA1 -> STN1NK60ZL; footprint Package_TO_SOT_SMD:SOT-223-3_TabPin2 -> OMNIXIE:SOT-223-MiddlePinDrain
- R10, R16: value 10k -> 30K
- R3: footprint Resistor_SMD:R_0603_1608Metric -> Resistor_SMD:R_0603_1608Metric_Pad0.98x0.95mm_HandSolder
- TP10: now fitted; now in the parts list
Connections:
- net +3V3: now also TP17.1
- net +3V3_JUMP: now also TP24.1
- net +5V: now also TP18.1, TP21.1
- net CATH0: now also J7.1 (Pin_1)
- net CATH1: now also J7.2 (Pin_2)
- net CATH2: now also J7.3 (Pin_3)
- net CATH3: now also J7.4 (Pin_4)
- net CATH4: now also J7.5 (Pin_5)
- net CATH5: now also J7.6 (Pin_6)
- net CATH6: now also J7.7 (Pin_7)
- net CATH7: now also J7.8 (Pin_8)
- net CATH8: now also J7.9 (Pin_9)
- net CATH9: now also J7.10 (Pin_10)
- net CATHAUX: now also J7.12 (Pin_12)
- net CATHDP: now also J7.11 (Pin_11)
- net D+: now also TP20.1
- net D-: now also TP19.1
- net GND: now also J4.SH (SHIELD), Q12.3 (S), J7.13 (Pin_13), J7.14 (Pin_14), TP25.1; no longer J4.S1 (SHIELD), Q12.2 (S)
- net HIGHVOLTAGE: now also J7.15 (Pin_15), J7.16 (Pin_16)
- net I2C_SCL: now also U1.9 (PC2/SCL/URTS/T1BKIN/AETR/T2CH2/T1ETR), TP15.1, TP22.1; no longer U1.10 (PC3/T1CH3/T1CHIN/UCTS)
- net I2C_SDA: now also U1.8 (PC1/SDA/NSS/T2CH4/T2CH1ETR/T1BKIN/URX), TP16.1, TP23.1; no longer U1.9 (PC2/SCL/URTS/T1BKIN/AETR/T2CH2/T1ETR)
- net PC1: no longer U1.8 (PC1/SDA/NSS/T2CH4/T2CH1ETR/T1BKIN/URX)
- net at T1.4: now also Q12.2 (D); no longer Q12.3 (D)
- new net PC3: U1.10 (PC3/T1CH3/T1CHIN/UCTS)
Other:
- note removed: ">.< Add redundant path for signals if connector would be very hard to probe on."
- note removed: ">.< Board is WAY TOO SMALL for a first development prototype"
- note removed: ">.< Footprint pin assignments wrong for flyback switching MOSFET"
- note removed: ">.< I am not confident that I will be able to drive the MOSFET I chose correctly with a 3.3V PWM"
- note removed: ">.< LEDs are TOO BRIGHT. Increase resistance"
- note removed: ">.< Might be worth it to get SMT test loops if space allows"
- note removed: ">.< Pins 8 9 and 10 wrong pinout. I2C SDA and SCL defined on wrong pins."
- note removed: ">.< Silkscreen WAY TOO SMALL to be easily legible from a reasonable distance"
- moved on the sheet: C4, FID10, FID11, FID12, FID13, FID14, FID15, FID9, J5, J8, JP10, JP11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

Commit message: board bringup starting now
Parts:
- removed TP15, TP16, TP21: 5005, TestPoint:TestPoint_Keystone_5005-5009_Compact, symbol Connector:TestPoint
- added R17: JUMPER, Resistor_SMD:R_0805_2012Metric, symbol cnixxie:R
- C1, C2, C3, C4, C5, D3, R10, R11, R12, R13, R14, R15, R16, R3, R5, R6, R7, R8, R9: KiLib_Generator (none) -> SMD_2terminal_chip_molded
- J1, J5, J6, J7: KiLib_Generator (none) -> connector/pin_header_socket
- J2, J3: KiLib_Generator (none) -> connector/SMD_single_row_plus_mounting_pad
- U1: KiLib_Generator (none) -> package/no_lead
Connections:
- net PC1 is gone; now on net PC6: J1.4 (Pin_4)
- net +3V3: now also J5.3 (Pin_3), TP24.1
- net +3V3_JUMP: no longer J5.3 (Pin_3), TP24.1
- net CATH5: no longer J7.6 (Pin_6)
- net CATH7: no longer J7.8 (Pin_8)
- net CATH8: no longer J7.9 (Pin_9)
- net CATH9: no longer J7.10 (Pin_10)
- net CATHAUX: no longer J7.12 (Pin_12)
- net CATHDP: no longer J7.11 (Pin_11)
- net HV_SW: now also R17.1; no longer Q12.1 (G), R12.1, TP14.1
- net PA1: now also J1.10 (Pin_10); no longer J1.8 (Pin_8)
- net PA2: now also J1.9 (Pin_9); no longer J1.7 (Pin_7)
- net PC0: now also J1.7 (Pin_7); no longer J1.5 (Pin_5)
- net PC3: now also J1.6 (Pin_6)
- net PC5: now also J1.5 (Pin_5); no longer J1.3 (Pin_3)
- net PC6: no longer J1.2 (Pin_2)
- net PD0: now also J1.8 (Pin_8); no longer J1.6 (Pin_6)
- net PD2: now also J1.3 (Pin_3); no longer J1.1 (Pin_1)
- net PD6: now also J1.1 (Pin_1); no longer J1.10 (Pin_10)
- net PD7: now also J1.2 (Pin_2); no longer J1.9 (Pin_9)
- new net: Q12.1 (G), R12.1, R17.2, TP14.1
- no-connect marks 10 -> 20
Other:
- note removed: ">.< Use a horizontal mount USB-C or at least put the vertical USB-C on the same side as the header pins and test loops so that on the bench you don't have wires bending up and around from the bottom of the board when the USB-C is plugged in"
- note removed: "REDLINE NOTES"
